File: Hardware/SNVA717_V1.1/SNVA717_V1.1.kicad_pcb (KiCad board)
At the start: 2 copper layers, 54.6 x 12.7 mm, 20 parts, among them Q1 MMBT3906, Q2 AO3401A

Commit message: Fix Q1
Parts:
- moved Q1 1.20 mm to (82.4, 50.8), turned to -90 degrees
Connections:
- Q1 pad 2: Net-(D3-A) -> Net-(D1-K)
- Q1 pad 3: Net-(D1-K) -> Net-(D3-A)
Routing:
- net Net-(D2-K): track 4.13 -> 6.61 mm
- net Net-(D3-A): track 20.8 -> 22.3 mm
Changed lines of the file:
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@@
 	(footprint "Package_TO_SOT_SMD:SOT-23"
 		(layer "F.Cu")
-		(at 82.4 49.6 90)
+		(at 82.4 50.8 -90)
 		(descr "SOT, 3 Pin (JEDEC TO-236 Var AB https://www.jedec.org/document_search?search_api_views_fulltext=TO-236), generated with kicad-footprint-generator ipc_gullwing_generator.py")
 		(tags "SOT TO_SOT_SMD")
@@
 		(attr smd)
 		(fp_line
-			(start 0 -1.56)
-			(end 0.65 -1.56)
+			(start 0 1.56)
+			(end -0.65 1.56)
 			(stroke
 				(width 0.12)
@@
 		)
 		(fp_line
-			(start 0 -1.56)
-			(end -0.65 -1.56)
+			(start 0 1.56)
+			(end 0.65 1.56)
 			(stroke
 				(width 0.12)
@@
 		)
 		(fp_line
-			(start 0 1.56)
-			(end 0.65 1.56)
+			(start 0 -1.56)
+			(end -0.65 -1.56)
 			(stroke
 				(width 0.12)
@@
 		)
 		(fp_line
-			(start 0 1.56)
-			(end -0.65 1.56)
+			(start 0 -1.56)
+			(end 0.65 -1.56)
 			(stroke
 				(width 0.12)
@@
 		)
 		(fp_line
-			(start 1.92 -1.7)
-			(end -1.92 -1.7)
+			(start -1.92 1.7)
+			(end 1.92 1.7)
 			(stroke
 				(width 0.05)
@@
 		)
 		(fp_line
-			(start -1.92 -1.7)
-			(end -1.92 1.7)
+			(start 1.92 1.7)
+			(end 1.92 -1.7)
 			(stroke
 				(width 0.05)
@@
 		)
 		(fp_line
-			(start 1.92 1.7)
-			(end 1.92 -1.7)
+			(start -1.92 -1.7)
+			(end -1.92 1.7)
 			(stroke
 				(width 0.05)
@@
 		)
 		(fp_line
-			(start -1.92 1.7)
-			(end 1.92 1.7)
+			(start 1.92 -1.7)
+			(end -1.92 -1.7)
 			(stroke
 				(width 0.05)
@@
 		)
 		(fp_line
-			(start 0.65 -1.45)
-			(end 0.65 1.45)
+			(start -0.65 1.45)
+			(end -0.65 -1.125)
 			(stroke
 				(width 0.1)
@@
 		)
 		(fp_line
-			(start -0.325 -1.45)
-			(end 0.65 -1.45)
+			(start 0.65 1.45)
+			(end -0.65 1.45)
 			(stroke
 				(width 0.1)
@@
 		)
 		(fp_line
-			(start 0.65 1.45)
-			(end -0.65 1.45)
+			(start -0.325 -1.45)
+			(end 0.65 -1.45)
 			(stroke
 				(width 0.1)
@@
 		)
 		(fp_line
-			(start -0.65 1.45)
-			(end -0.65 -1.125)
+			(start 0.65 -1.45)
+			(end 0.65 1.45)
 			(stroke
 				(width 0.1)
@@
 		)
 		(pad "1" smd roundrect
-			(at -0.9375 -0.95 90)
+			(at -0.9375 -0.95 270)
 			(size 1.475 0.6)
 			(layers "F.Cu" "F.Paste" "F.Mask")
@@
 		)
 		(pad "2" smd roundrect
-			(at -0.9375 0.95 90)
+			(at -0.9375 0.95 270)
 			(size 1.475 0.6)
 			(layers "F.Cu" "F.Paste" "F.Mask")
 			(roundrect_rratio 0.25)
-			(net 3 "Net-(D3-A)")
+			(net 2 "Net-(D1-K)")
 			(pinfunction "E")
 			(pintype "passive")
 		)
 		(pad "3" smd roundrect
-			(at 0.9375 0 90)
+			(at 0.9375 0 270)
 			(size 1.475 0.6)
 			(layers "F.Cu" "F.Paste" "F.Mask")
 			(roundrect_rratio 0.25)
-			(net 2 "Net-(D1-K)")
+			(net 3 "Net-(D3-A)")
 			(pinfunction "C")
 			(pintype "passive")
@@
 		(tags "SOT TO_SOT_SMD")
 		(property "Reference" "Q2"
-			(at 0 -2.4 360)
+			(at 0 -2.4 0)
 			(layer "F.SilkS")
 			(hide yes)
@@
 		)
 		(property "Value" "AO3401A"
-			(at 0 2.4 360)
+			(at 0 2.4 0)
 			(layer "F.Fab")
 			(effects
@@
 		)
 		(property "Footprint" "Package_TO_SOT_SMD:SOT-23"
-			(at 0 0 360)
+			(at 0 0 0)
 			(layer "F.Fab")
 			(hide yes)
@@
 		)
 		(property "Datasheet" "http://www.aosmd.com/pdfs/datasheet/AO3401A.pdf"
-			(at 0 0 360)
+			(at 0 0 0)
 			(layer "F.Fab")
 			(hide yes)
@@
 		)
 		(property "Description" "-4.0A Id, -30V Vds, P-Channel MOSFET, SOT-23"
-			(at 0 0 360)
+			(at 0 0 0)
 			(layer "F.Fab")
 			(hide yes)
@@
 		)
 		(fp_text user "${REFERENCE}"
-			(at 0 0 360)
+			(at 0 0 0)
 			(layer "F.Fab")
 			(effects
@@
 		(tags "resistor")
 		(property "Reference" "R5"
-			(at 0 -1.17 360)
+			(at 0 -1.17 0)
 			(layer "F.SilkS")
 			(hide yes)
@@
 		)
 		(property "Value" "10.2K"
-			(at 0 1.17 360)
+			(at 0 1.17 0)
 			(layer "F.Fab")
 			(effects
@@
 		)
 		(fp_text user "${REFERENCE}"
-			(at 0 0 360)
+			(at 0 0 0)
 			(layer "F.Fab")
 			(effects
@@
 		(tags "Diode SMA (DO-214AC)")
 		(property "Reference" "D1"
-			(at 0 -2.5 360)
+			(at 0 -2.5 0)
 			(layer "F.SilkS")
 			(hide yes)
@@
 		)
 		(property "Value" "US1M"
-			(at 0 2.6 360)
+			(at 0 2.6 0)
 			(layer "F.Fab")
 			(effects
@@
 		)
 		(fp_text user "${REFERENCE}"
-			(at 0 -2.5 360)
+			(at 0 -2.5 0)
 			(layer "F.Fab")
 			(effects
@@
 	)
 	(segment
+		(start 86.8 50.4625)
+		(end 86.7275 50.39)
+		(width 0.3)
+		(layer "F.Cu")
+		(net 3)
+	)
+	(segment
 		(start 82.9 46.925)
 		(end 81.4 45.425)
@@
 	)
 	(segment
-		(start 86.8 50.4625)
-		(end 83.425 50.4625)
+		(start 84.6 50.39)
+		(end 83.2525 51.7375)
 		(width 0.3)
 		(layer "F.Cu")
@@
 	)
 	(segment
-		(start 83.425 50.4625)
-		(end 83.35 50.5375)
+		(start 86.7275 50.39)
+		(end 84.6 50.39)
 		(width 0.3)
 		(layer "F.Cu")
@@
 	)
 	(segment
+		(start 83.2525 51.7375)
+		(end 82.4 51.7375)
+		(width 0.3)
+		(layer "F.Cu")
+		(net 3)
+	)
+	(segment
 		(start 86.89 50.3725)
 		(end 86.8 50.4625)
@@
 	)
 	(segment
-		(start 80.9125 50)
-		(end 81.45 50.5375)
+		(start 80.404 50.904)
+		(end 81.79221 50.904)
 		(width 0.3)
 		(layer "F.Cu")
@@
 	)
 	(segment
-		(start 78.89 50.61)
-		(end 79.5 50)
+		(start 82.83371 49.8625)
+		(end 83.35 49.8625)
+		(width 0.3)
+		(layer "F.Cu")
+		(net 4)
+	)
+	(segment
+		(start 81.79221 50.904)
+		(end 82.83371 49.8625)
 		(width 0.3)
 		(layer "F.Cu")
@@
 	(segment
 		(start 79.5 50)
-		(end 80.9125 50)
+		(end 80.404 50.904)
+		(width 0.3)
+		(layer "F.Cu")
+		(net 4)
+	)
+	(segment
+		(start 78.89 50.61)
+		(end 79.5 50)
 		(width 0.3)
 		(layer "F.Cu")
@@
 		(polygon
 			(pts
-				(xy 75.4 48.5) (xy 76 49) (xy 81.3 49) (xy 82.133333 49.7) (xy 82.766668 49.7) (xy 82.875001 49.6)
+				(xy 75.4 48.5) (xy 76 49) (xy 80.6 49) (xy 81.433333 49.7) (xy 82.766668 49.7) (xy 82.875001 49.6)
 				(xy 84.842855 49.6) (xy 85.4 48.3) (xy 85.4 47.3) (xy 85.2 47.1) (xy 81.8 47.1) (xy 79.6 44.9) (xy 76.2 44.9)
 				(xy 75.4 45.749438)
